File: VTOL.kicad_pcb (KiCad board)
At the start: 2 copper layers, 45 parts, among them J1 Conn_01x06_Pin, J2 Conn_01x06_Pin, J3 Conn_01x04_Pin, J5 USB_C_Receptacle_USB2.0_16P, J6 Conn_01x02_Pin, J7 Conn_01x06_Pin, SW1 RESET, SW2 RESET, U1 DS18B20, U2 SEN0460, U3 Si7021-A20, U4 ESP32-S3-WROOM-1, U5 USBLC6-2SC6, U6 AMS1117-3.3

Commit message: barely finished pcb
Parts:
- moved H6 99.1 mm to (227.9, 59.1)
- moved H3 92.9 mm to (180.0, 22.7)
- moved H4 89.4 mm to (208.1, 58.9)
- moved H1 82.9 mm to (114.9, 23.3)
- moved H8 79.7 mm to (228.4, 87.9)
- moved F2 72.2 mm to (121.5, 70.0)
- moved FB2 72.2 mm to (121.5, 75.9)
- moved D2 70.9 mm to (127.9, 70.8), turned to 180 degrees
- moved U3 70.5 mm to (226.6, 75.3), turned to -90 degrees
- moved U5 69.1 mm to (134.3, 63.7)
- moved C2 60.5 mm to (132.2, 101.6), turned to 180 degrees
- moved J5 59.0 mm to (122.5, 63.3), turned to -90 degrees
- moved H7 58.3 mm to (208.5, 88.0)
- moved D3 55.3 mm to (137.1, 89.2), turned to 180 degrees
- moved R1 53.8 mm to (126.2, 90.0), turned to 90 degrees
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Routing:
- net +3.3V: track 0.00 -> 161.6 mm
- net /BOOT: track 0.00 -> 75.0 mm, vias 0 -> 6
- net /EN: track 0.00 -> 73.9 mm, vias 0 -> 2
- net /SCL: track 0.00 -> 63.9 mm, vias 0 -> 4
- net /TEMP_DATA: track 0.00 -> 62.6 mm, vias 0 -> 2
- net /SDA: track 0.00 -> 57.1 mm, vias 0 -> 4
- net /CC1: track 0.00 -> 41.2 mm, vias 0 -> 2
- net Net-(D1-K): track 0.00 -> 39.9 mm, vias 0 -> 2
- net +5V: track 0.00 -> 38.5 mm, vias 0 -> 2
- net /PI_TX: track 0.00 -> 35.0 mm, vias 0 -> 2
- net +BATT: track 0.00 -> 34.2 mm, vias 0 -> 2
- net /PI_3V3: track 0.00 -> 32.0 mm
- net /PI_RX: track 0.00 -> 30.2 mm, vias 0 -> 2
- net /CC2: track 0.00 -> 27.8 mm
- net /D-: track 0.00 -> 24.2 mm
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- added copper zone on B.Cu, net GND
- added copper zone on F.Cu, net GND
Other:
- board outline added: 124.9 x 103.9 mm
- copper layers 2 -> 4
