File: VTOL.kicad_pcb (KiCad board)
At the start: 4 copper layers, 76.5 x 104 mm, 36 parts, among them J10 I2C header, J5 USB_C_Receptacle_USB2.0_16P, J6 Conn_01x02_Pin, J7 Pi UART, J8 SEN66, J9 I2C header, SW1 RESET, SW2 BOOT, SW3 SW_SPDT, U4 ESP32-S3-WROOM-1, U5 USBLC6-2SC6, U6 AP7361C-33ER-13, U7 R-78E5.0-1.0

Commit message: Add INA226 power monitor, finish part selection, clear PCB
- Schematic: INA226 (U1) + 20m shunt (R3) + C2 on the 5V rail, I2C 0x44
- Sections boxed and titled; on-sheet notes removed
- Footprint and DigiKey part # set for every part
- J8 -> Molex 0702461201 with 1.1mm-drill IDC 2x06 footprint
- D6 -> red LED on 3.3V
- PCB cleared for re-layout
Parts:
- removed C1, C11, C12, C5: 10u 25V, Capacitor_SMD:C_0805_2012Metric_Pad1.18x1.45mm_HandSolder
- removed C10, C4: 0.1u 50V, Capacitor_SMD:C_0603_1608Metric_Pad1.08x0.95mm_HandSolder
- removed C13: 47u 35V, Capacitor_SMD:CP_Elec_6.3x5.8
- removed C14: 47u 10V, Capacitor_SMD:C_1206_3216Metric_Pad1.33x1.80mm_HandSolder
- removed C3: 1u 50V, Capacitor_SMD:C_0603_1608Metric_Pad1.08x0.95mm_HandSolder
- removed C7: 10u 50V, Capacitor_SMD:C_1206_3216Metric_Pad1.33x1.80mm_HandSolder
- removed D1: SMF5.0A, Diode_SMD:D_SOD-123F
- removed F1: 1A, Fuse:Fuse_1206_3216Metric_Pad1.42x1.75mm_HandSolder
- removed F2: 0.75A 24V, Fuse:Fuse_1812_4532Metric_Pad1.30x3.40mm_HandSolder
- removed H1, H2, H3, H5: MountingHole, MountingHole:MountingHole_3.2mm_M3_Pad_Via
- removed J10, J9: I2C header, Connector_PinHeader_2.54mm:PinHeader_1x04_P2.54mm_Vertical
- removed J5: USB_C_Receptacle_USB2.0_16P, VTOL_parts:USB_C_Receptacle_GCT_USB4105-GF-A_16P_TopMnt_Horizontal_S1
- removed J6: Conn_01x02_Pin, Connector_JST:JST_PH_S2B-PH-K_1x02_P2.00mm_Horizontal
- removed J7: Pi UART, Connector_PinHeader_2.54mm:PinHeader_1x03_P2.54mm_Vertical
- removed J8: SEN66, Connector_JST:JST_GH_BM06B-GHS-TBT_1x06-1MP_P1.25mm_Vertical
- removed R1, R2: 10k, Resistor_SMD:R_0603_1608Metric_Pad0.98x0.95mm_HandSolder
- removed R3, R4: 4.7k, Resistor_SMD:R_0603_1608Metric_Pad0.98x0.95mm_HandSolder
- removed R5, R9: 5.1k, Resistor_SMD:R_0603_1608Metric_Pad0.98x0.95mm_HandSolder
- removed SW1: RESET, Button_Switch_SMD:SW_SPST_PTS645Sx43SMTR92
- removed SW2: BOOT, Button_Switch_SMD:SW_SPST_PTS645Sx43SMTR92
- removed SW3: SW_SPDT, VTOL_parts:SW_Slide_SPDT_RightAngle_CK_1101M2S3AQE2
- removed U4: ESP32-S3-WROOM-1, VTOL_parts:ESP32-S3-WROOM-1_Via0.3mm
- removed U5: USBLC6-2SC6, Package_TO_SOT_SMD:SOT-23-6
- removed U6: AP7361C-33ER-13, Package_TO_SOT_SMD:SOT-223-3_TabPin2
- removed U7: R-78E5.0-1.0, Converter_DCDC:Converter_DCDC_RECOM_R-78E-0.5_THT
Routing:
- net /SCL: track 95.4 -> 0.00 mm, vias 3 -> 0
- net /SDA: track 79.1 -> 0.00 mm, vias 2 -> 0
- net GND: track 40.7 -> 0.00 mm, vias 25 -> 0
- net VBUS: track 39.9 -> 0.00 mm, vias 2 -> 0
- net /ESP_TX: track 31.6 -> 0.00 mm, vias 1 -> 0
- net /ESP_RX: track 27.6 -> 0.00 mm
- net /BATT_5V: track 25.2 -> 0.00 mm
- net +BATT: track 23.4 -> 0.00 mm
- net /EN: track 22.4 -> 0.00 mm
- net /BOOT: track 20.6 -> 0.00 mm
- net /D+: track 20.2 -> 0.00 mm
- net +3.3V: track 18.8 -> 0.00 mm, vias 13 -> 0
- net /USB_D+: track 15.6 -> 0.00 mm, vias 2 -> 0
- net /USB_D-: track 12.3 -> 0.00 mm
- net /5V_FUSED: track 11.8 -> 0.00 mm
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- removed copper zone on In2.Cu, net +3.3V
- removed copper zone on B.Cu, net GND
- removed copper zone on F.Cu, net GND
- removed copper zone on In1.Cu, net GND
Other:
- board outline removed
- board text removed: "3V3"
- board text removed: "GND"
- board text removed: "SCL"
- board text removed: "SDA"
