File: VTOL.kicad_sch (KiCad schematic)
At the start: 45 parts, among them J1 Conn_01x06_Pin, J2 Conn_01x06_Pin, J3 Conn_01x04_Pin, J5 USB_C_Receptacle_USB2.0_16P, J6 Conn_01x02_Pin, J7 Conn_01x06_Pin, SW1 RESET, SW2 RESET, U1 DS18B20, U2 SEN0460, U3 Si7021-A20, U4 ESP32-S3-WROOM-1, U5 USBLC6-2SC6, U6 AMS1117-3.3

Commit message: Snapshot before PCB cleanup/re-route
Schematic fixes (C1/C5 polarity, SEN0460 on 5V_FUSED, decoupling C8-C11, labels) and current messy PCB, saved so the re-layout can be reverted.

Co-Authored-By: Claude Opus 5.5 <noreply@anthropic.com>
Parts:
- removed D2, D3: 1A, symbol Device:D_Schottky
- removed F2: 500mA, symbol Device:Polyfuse
- removed FB1, FB2: FerriteBead, symbol Device:FerriteBead
- added C10, C8, C9: 0.1u, Capacitor_SMD:C_0603_1608Metric_Pad1.08x0.95mm_HandSolder, symbol Device:C
- added C11: 10u, Capacitor_SMD:C_0805_2012Metric_Pad1.18x1.45mm_HandSolder, symbol Device:C
- added SW3: SW_SPDT, Button_Switch_SMD:Nidec_Copal_CAS-120A, symbol Switch:SW_SPDT
- C1: footprint (none) -> Capacitor_Tantalum_SMD:CP_EIA-3528-21_Kemet-B_HandSolder; symbol Device:C -> Device:C_Polarized
- C2, C3, C4, C6: footprint (none) -> Capacitor_SMD:C_0603_1608Metric_Pad1.08x0.95mm_HandSolder
- C5: value 10u -> 22u; footprint (none) -> Capacitor_Tantalum_SMD:CP_EIA-3528-21_Kemet-B; symbol Device:C -> Device:C_Polarized
- C7: footprint (none) -> Capacitor_Tantalum_SMD:CP_EIA-3528-21_Kemet-B
- F1: footprint (none) -> Fuse:Fuse_1206_3216Metric_Pad1.42x1.75mm_HandSolder
- H1, H2, H3, H4, H5, H6, H7, H8: footprint (none) -> MountingHole:MountingHole_3.2mm_M3_Pad_Via
- J1, J2: footprint (none) -> Connector_JST:JST_SH_SM06B-SRSS-TB_1x06-1MP_P1.00mm_Horizontal
- J3, U2: footprint (none) -> Connector_PinHeader_2.54mm:PinHeader_1x04_P2.54mm_Vertical
- J5: footprint (none) -> Connector_USB:USB_C_Receptacle_HRO_TYPE-C-31-M-12
- J6: footprint (none) -> Connector_PinHeader_1.00mm:PinHeader_1x02_P1.00mm_Horizontal
- J7: footprint (none) -> Connector_PinHeader_2.54mm:PinHeader_1x06_P2.54mm_Vertical
- R1, R2, R3, R4, R5, R6, R7, R8, R9: footprint (none) -> Resistor_SMD:R_0603_1608Metric_Pad0.98x0.95mm_HandSolder
- SW1: footprint (none) -> Button_Switch_SMD:SW_SPST_PTS645Sx43SMTR92
- SW2: value RESET -> BOOT; footprint (none) -> Button_Switch_SMD:SW_SPST_PTS645Sx43SMTR92
Connections:
- net +3.3V: now also C10.1, C11.1, C8.1, C9.1; no longer U2.1 (VIN)
- net +5V: now also SW3.2 (B); no longer C4.2, U5.5 (VBUS)
- net +BATT: now also SW3.1 (A)
- net GND: now also C1.2, C10.2, C11.2, C8.2, C9.2; no longer C1.1
- net 5V_FUSED: now reaches J2.6 (Pin_6)
- net 5V_FUSED: now also C1.1, C2.2, D1.1 (K), F1.2, J1.6 (Pin_6), U2.1 (VIN), U6.3 (VI)
- net VBUS: now reaches J5.A4 (VBUS), J5.A9 (VBUS), J5.B4 (VBUS), J5.B9 (VBUS)
- net VBUS: now also C4.2, U5.5 (VBUS), SW3.3 (C)
- net PI_RX renamed ESP_RX
- net PI_TX renamed ESP_TX
- no-connect marks 32 -> 30

Commit message: Rework power, sensors and PCB layout; add DigiKey BOM
- Power: 4S LiPo input (J6 -> F2 polyfuse -> R-78E 5V buck) with hot-plug
  damping cap (C13), USB/battery select switch SW3, AP7361C LDO with
  ceramic caps.
- Sensors: SEN66 (J8) replaces SEN0460/Si7021/DS18B20; two I2C headers.
- Pi link reduced to a 3-pin UART; camera pass-through removed.
- PCB: re-placed by function, 4-layer (GND + 3V3 planes), rerouted,
  DigiKey footprint swaps in the VTOL_parts library, sub-board removed.
- Schematic tidy: decoupling caps grouped on shared rails; drop redundant
  C2/C6 0.1u caps.
- BOM_digikey.csv for DigiKey BOM Manager.

Co-Authored-By: Claude Opus 5.5 <noreply@anthropic.com>
Parts:
- removed C2, C6, C8, C9: 0.1u, Capacitor_SMD:C_0603_1608Metric_Pad1.08x0.95mm_HandSolder, symbol Device:C
- removed H4, H6, H7, H8: MountingHole, MountingHole:MountingHole_3.2mm_M3_Pad_Via, symbol Mechanical:MountingHole
- removed J1, J2: Conn_01x06_Pin, Connector_JST:JST_SH_SM06B-SRSS-TB_1x06-1MP_P1.00mm_Horizontal, symbol Connector:Conn_01x06_Pin
- removed J3: Conn_01x04_Pin, Connector_PinHeader_2.54mm:PinHeader_1x04_P2.54mm_Vertical, symbol Connector:Conn_01x04_Pin
- removed R6, R7, R8: 4.7k, Resistor_SMD:R_0603_1608Metric_Pad0.98x0.95mm_HandSolder, symbol Device:R
- removed U1: DS18B20, Package_TO_SOT_THT:TO-92_Inline, symbol Sensor_Temperature:DS18B20
- removed U2: SEN0460, Connector_PinHeader_2.54mm:PinHeader_1x04_P2.54mm_Vertical, symbol Sensor_Symbols:SEN0460
- removed U3: Si7021-A20, Package_DFN_QFN:DFN-6-1EP_3x3mm_P1mm_EP1.5x2.4mm, symbol Sensor_Humidity:Si7021-A20
- added C12: 10u 25V, Capacitor_SMD:C_0805_2012Metric_Pad1.18x1.45mm_HandSolder, symbol Device:C
- added C13: 47u 35V, Capacitor_SMD:CP_Elec_6.3x5.8, symbol Device:C_Polarized
- added C14: 47u 10V, Capacitor_SMD:C_1206_3216Metric_Pad1.33x1.80mm_HandSolder, symbol Device:C
- added F2: 0.75A 24V, Fuse:Fuse_1812_4532Metric_Pad1.30x3.40mm_HandSolder, symbol Device:Polyfuse
- added J10, J9: I2C header, Connector_PinHeader_2.54mm:PinHeader_1x04_P2.54mm_Vertical, symbol Connector:Conn_01x04_Pin
- added J8: SEN66, Connector_JST:JST_GH_BM06B-GHS-TBT_1x06-1MP_P1.25mm_Vertical, symbol Connector:Conn_01x06_Pin
- added U7: R-78E5.0-1.0, Converter_DCDC:Converter_DCDC_RECOM_R-78E-0.5_THT, symbol Converter_DCDC:R-78E5.0-1.0
- C1: value 100u -> 10u 25V; footprint Capacitor_Tantalum_SMD:CP_EIA-3528-21_Kemet-B_HandSolder -> Capacitor_SMD:C_0805_2012Metric_Pad1.18x1.45mm_HandSolder; symbol Device:C_Polarized -> Device:C
- C10, C4: value 0.1u -> 0.1u 50V
- C11: value 10u -> 10u 25V
- C3: value 0.1u -> 1u 50V
- C5: value 22u -> 10u 25V; footprint Capacitor_Tantalum_SMD:CP_EIA-3528-21_Kemet-B -> Capacitor_SMD:C_0805_2012Metric_Pad1.18x1.45mm_HandSolder; symbol Device:C_Polarized -> Device:C
- C7: value 100u -> 10u 50V; footprint Capacitor_Tantalum_SMD:CP_EIA-3528-21_Kemet-B -> Capacitor_SMD:C_1206_3216Metric_Pad1.33x1.80mm_HandSolder; symbol Device:C_Polarized -> Device:C
- D1: value PTVS5V0Z1USK -> SMF5.0A; footprint Diode_SMD:Nexperia_DSN1608-2_1.6x0.8mm -> Diode_SMD:D_SOD-123F
- J5: footprint Connector_USB:USB_C_Receptacle_HRO_TYPE-C-31-M-12 -> VTOL_parts:USB_C_Receptacle_GCT_USB4105-GF-A_16P_TopMnt_Horizontal_S1
- J6: footprint Connector_PinHeader_1.00mm:PinHeader_1x02_P1.00mm_Horizontal -> Connector_JST:JST_PH_S2B-PH-K_1x02_P2.00mm_Horizontal
- J7: value Conn_01x06_Pin -> Pi UART; footprint Connector_PinHeader_2.54mm:PinHeader_1x06_P2.54mm_Vertical -> Connector_PinHeader_2.54mm:PinHeader_1x03_P2.54mm_Vertical; symbol Connector:Conn_01x06_Pin -> Connector:Conn_01x03_Pin
- SW3: footprint Button_Switch_SMD:Nidec_Copal_CAS-120A -> VTOL_parts:SW_Slide_SPDT_RightAngle_CK_1101M2S3AQE2
- U4: footprint RF_Module:ESP32-S3-WROOM-1 -> VTOL_parts:ESP32-S3-WROOM-1_Via0.3mm
- U6: value AMS1117-3.3 -> AP7361C-33ER-13
Connections:
- net CAM_SDA is gone; now on net GND: J7.3 (Pin_3)
- net +3.3V: now also C14.1, J10.2 (Pin_2), J8.1 (Pin_1), J8.6 (Pin_6), J9.2 (Pin_2)
- net +BATT: now also C13.1, F2.2, U7.1 (IN); no longer J6.1 (Pin_1), SW3.1 (A)
- net GND: now also C12.2, C13.2, C14.2, J10.1 (Pin_1), J8.2 (Pin_2), J8.5 (Pin_5), J9.1 (Pin_1), U7.2 (GND); no longer J7.6 (Pin_6)
- net SCL: now also J10.4 (Pin_4), J8.4 (Pin_4), J9.4 (Pin_4)
- net SDA: now also J10.3 (Pin_3), J8.3 (Pin_3), J9.3 (Pin_3)
- removed net CAM_SCL: J7.4 (Pin_4)
- removed net PI_3V3: J7.5 (Pin_5)
- net TEMP_DATA: no longer names the net of U4.4 (IO4)
- new net BATT_5V: C12.1, SW3.1 (A), U7.3 (OUT)
- new net BATT_IN: F2.1, J6.1 (Pin_1)
- no-connect marks 30 -> 31
Other:
- note added: "Air quality + temp/RH (SEN66, J8) I2C expansion headers (J9, J10)"
- note added: "I2C BUS PULL-UPS"
- note added: "RASPBERRY PI UART LINK (J7) Camera plugs into the Pi directly"
- note added: "SENSOR CONNECTORS"
- note removed: "CAMERA CONNECT PASS THROUGH (MLX90640 DEV BOARD)"
- note removed: "I2C BUS + SINGLE DATA LINE FOR TEMP"
- note removed: "SENSOR MODULE"
- note removed: "Temperature Sensor, Air Quality, LiDAR/Ultrasonic Distance Sensor"
- moved on the sheet: C10, C11, D1, F1, J6, U6
